File: DAC/DAC-peripherals/level_shifter_parallell_sch.kicad_sch (KiCad schematic)
At the start: 1 part, among them J3 Conn_01x10_Female

Commit message: improved PCB again again
Parts:
- renumbered J3 to J4
Changed lines of the file:
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@@
   (symbol (lib_id "Connector:Conn_01x10_Female") (at 101.6 90.17 180) (unit 1)
     (in_bom yes) (on_board yes) (fields_autoplaced)
-    (property "Reference" "J3" (id 0) (at 102.235 72.39 0))
+    (property "Reference" "J4" (id 0) (at 102.235 72.39 0))
     (property "Value" "Conn_01x10_Female" (id 1) (at 102.235 74.93 0))
     (property "Footprint" "Connector_PinSocket_2.54mm:PinSocket_1x10_P2.54mm_Vertical" (id 2) (at 101.6 90.17 0)
