File: DAC/DAC-peripherals/DAC-peripherals.kicad_sch (KiCad schematic)
At the start: 13 parts, among them IC1 THS8135PHP, J1 Conn_01x04_Female, J2 Conn_01x02_Female, J6 Conn_01x01_Female, J7 Conn_01x01_Female, U1 SN74LV1T34DBV

Commit message: improved PCB design
Parts:
- removed C1: C, Capacitor_SMD:C_0805_2012Metric, symbol pspice:C
- removed C2, C3: 0.1u, Capacitor_SMD:C_0805_2012Metric, symbol pspice:C
- removed J1: Conn_01x04_Female, Connector_PinHeader_2.54mm:PinHeader_1x04_P2.54mm_Vertical, symbol Connector:Conn_01x04_Female
- removed J2: Conn_01x02_Female, Connector_PinHeader_2.54mm:PinHeader_1x02_P2.54mm_Vertical, symbol Connector:Conn_01x02_Female
- removed J6, J7: Conn_01x01_Female, Connector_PinHeader_2.54mm:PinHeader_1x01_P2.54mm_Vertical, symbol Connector:Conn_01x01_Female
- removed U1: SN74LV1T34DBV, Package_TO_SOT_SMD:SOT-23-5, symbol Logic_LevelTranslator:SN74LV1T34DBV
- added C1, C2, C3, C5, C6, C7: 100n, Capacitor_SMD:C_0603_1608Metric, symbol Device:C
- added C4: 4.7u, Capacitor_SMD:C_0603_1608Metric, symbol Device:C
- added J1, J2: Conn_01x03_Female, Connector_PinSocket_2.54mm:PinSocket_1x03_P2.54mm_Vertical, symbol Connector:Conn_01x03_Female
- added U1: LK112M18TR, Package_TO_SOT_SMD:SOT-23-5, symbol Regulator_Linear:LK112M18TR
- IC1: footprint QFP50P900X900X120-49N -> Package_QFP:TQFP-48-1EP_7x7mm_P0.5mm_EP5x5mm
- R1: value 37.5 -> 2k; footprint Resistor_SMD:R_0805_2012Metric -> Resistor_SMD:R_0603_1608Metric
- R2, R3, R4: value NC -> 75; footprint Resistor_SMD:R_0805_2012Metric -> Resistor_SMD:R_0603_1608Metric
Connections:
- net Level Shifter B/B1 is gone; now on net GND: IC1.9 (BCB1)
- net Level Shifter B/B10 is gone; now on net GND: IC1.10 (BCB0)
- net +1V8: now also IC1.11 (DVSS), IC1.23 (~{BLANK}), IC1.24 (~{SYNC}), IC1.25 (SYNC_T), C3.1, U1.4 (OUT); no longer IC1.12 (DVDD)
- net +3.3V: now also C1.1, C2.1, C4.1, C5.1, J1.3 (Pin_3), U1.1 (SHDN), U1.5 (IN); no longer IC1.23 (~{BLANK}), IC1.24 (~{SYNC}), IC1.25 (SYNC_T)
- net GND: now also IC1.12 (DVDD), IC1.49 (EP), R1.2, R2.2, R3.2, C1.2, C2.2, C3.2, C4.2, C6.2, C7.2, J1.1 (Pin_1), U1.2 (GND); no longer IC1.11 (DVSS), R1.1, R2.1, R3.1
- net at IC1.37 (VREF): now also C6.1
- net at IC1.39 (COMP): now also C5.2
- net out_x: now reaches R4.1
- net out_x: now also IC1.43 (ARPR), J2.1 (Pin_1); no longer IC1.41 (AGY)
- net CLK: now reaches IC1.26 (CLK)
- net out_i: now reaches IC1.45 (ABPB)
- net out_i: now also R2.1, J2.3 (Pin_3); no longer R2.2
- net FSADJ: now reaches IC1.38 (FSADJ)
- net FSADJ: now also R1.1; no longer R1.2
- net Level Shifter B/B2 renamed B1
- net Level Shifter B/B3 renamed B2
- net Level Shifter B/B4 renamed B3
- net Level Shifter B/B5 renamed B4
- net Level Shifter B/B6 renamed B5
- net Level Shifter B/B7 renamed B6
- net Level Shifter B/B8 renamed B7
- net Level Shifter B/B9 renamed B8
- net Level Shifter G/B1 renamed G2
- net Level Shifter G/B10 renamed G1
- net Level Shifter G/B2 renamed G3
- net Level Shifter G/B3 renamed G4
- net Level Shifter G/B4 renamed G5
- net Level Shifter G/B5 renamed G6
- net Level Shifter G/B6 renamed G7
- net Level Shifter G/B7 renamed G8
- net Level Shifter G/B8 renamed G9
- net Level Shifter G/B9 renamed G10
- net Level Shifter R/B1 renamed R1
- net Level Shifter R/B10 renamed R10
- net Level Shifter R/B2 renamed R2
- net Level Shifter R/B3 renamed R3
- net Level Shifter R/B4 renamed R4
- net Level Shifter R/B5 renamed R5
- net Level Shifter R/B6 renamed R6
- net Level Shifter R/B7 renamed R7
- net Level Shifter R/B8 renamed R8
- net Level Shifter R/B9 renamed R9
- new net: C7.1, U1.3 (Bypass)
- new net CLK_in: J1.2 (Pin_2)
- new net out_y: IC1.41 (AGY), J2.2 (Pin_2), R3.1
Other:
- removed sheet Level Shifter B
- removed sheet Level Shifter G
- removed sheet Level Shifter R
- added sheet level_shifter16 (level_shifter_sch.kicad_sch)
- added sheet level_shifter_parallell1 (level_shifter_parallell_sch.kicad_sch)
- added sheet level_shifter_parallell8 (level_shifter_parallell8_sch.kicad_sch)
- added sheet level_shifter_parallell_inv (level_shifter_parallell_inv_sch.kicad_sch)
- note added: "1.8 V LDO"
- note added: "Adjust depending on current output p.11 THS8135 datasheet"
- note added: "Close to AVDD"
- note added: "Close to DVDD"
- note added: "Optional termination resistors"

Commit message: improved PCB again again
Parts:
- removed J2: Conn_01x03_Female, Connector_PinSocket_2.54mm:PinSocket_1x03_P2.54mm_Vertical, symbol Connector:Conn_01x03_Female
- added J?: Conn_02x03_Odd_Even, symbol Connector_Generic:Conn_02x03_Odd_Even
Connections:
- net GND: now also J?.2 (Pin_2), J?.4 (Pin_4), J?.6 (Pin_6)
- net out_i: now also J?.5 (Pin_5)
- net out_x: now also J?.1 (Pin_1)
- net out_y: now also J?.3 (Pin_3)
Other:
- note added: "Optional GND connectors for each output"
Changed lines of the file:
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@@
   (junction (at 133.35 83.82) (diameter 0) (color 0 0 0 0)
   )
+  (junction (at 269.24 97.79) (diameter 0) (color 0 0 0 0)
+  )
   (junction (at 222.25 109.22) (diameter 0) (color 0 0 0 0)
   )
@@
   (junction (at 237.49 92.71) (diameter 0) (color 0 0 0 0)
   )
+  (junction (at 269.24 95.25) (diameter 0) (color 0 0 0 0)
+  )
   (junction (at 179.07 132.08) (diameter 0) (color 0 0 0 0)
   )
@@
   (junction (at 118.11 132.08) (diameter 0) (color 0 0 0 0)
   )
+  (wire (pts (xy 269.24 92.71) (xy 269.24 95.25))
+    (stroke (width 0) (type default) (color 0 0 0 0))
+  )
   (wire (pts (xy 179.07 130.81) (xy 179.07 132.08))
     (stroke (width 0) (type default) (color 0 0 0 0))
@@
     (stroke (width 0) (type default) (color 0 0 0 0))
   )
+  (polyline (pts (xy 266.7 91.44) (xy 271.78 91.44))
+    (stroke (width 0) (type default) (color 0 0 0 0))
+  )
   (wire (pts (xy 41.91 36.83) (xy 31.75 36.83))
     (stroke (width 0) (type default) (color 0 0 0 0))
@@
     (stroke (width 0) (type default) (color 0 0 0 0))
   )
+  (wire (pts (xy 269.24 97.79) (xy 269.24 100.33))
+    (stroke (width 0) (type default) (color 0 0 0 0))
+  )
   (wire (pts (xy 53.34 105.41) (xy 55.88 105.41))
     (stroke (width 0) (type default) (color 0 0 0 0))
@@
     (stroke (width 0) (type default) (color 0 0 0 0))
   )
+  (polyline (pts (xy 271.78 107.95) (xy 271.78 91.44))
+    (stroke (width 0) (type default) (color 0 0 0 0))
+  )
   (wire (pts (xy 182.88 82.55) (xy 182.88 81.28))
     (stroke (width 0) (type default) (color 0 0 0 0))
@@
     (stroke (width 0) (type default) (color 0 0 0 0))
   )
+  (polyline (pts (xy 266.7 91.44) (xy 266.7 107.95))
+    (stroke (width 0) (type default) (color 0 0 0 0))
+  )
   (wire (pts (xy 237.49 92.71) (xy 254 92.71))
     (stroke (width 0) (type default) (color 0 0 0 0))
@@
     (stroke (width 0) (type default) (color 0 0 0 0))
   )
+  (wire (pts (xy 269.24 95.25) (xy 269.24 97.79))
+    (stroke (width 0) (type default) (color 0 0 0 0))
+  )
   (polyline (pts (xy 58.42 17.78) (xy 58.42 45.72))
     (stroke (width 0) (type default) (color 0 0 0 0))
@@
     (stroke (width 0) (type default) (color 0 0 0 0))
   )
+  (wire (pts (xy 266.7 95.25) (xy 269.24 95.25))
+    (stroke (width 0) (type default) (color 0 0 0 0))
+  )
   (wire (pts (xy 213.36 97.79) (xy 222.25 97.79))
     (stroke (width 0) (type default) (color 0 0 0 0))
@@
     (stroke (width 0) (type default) (color 0 0 0 0))
   )
+  (wire (pts (xy 266.7 97.79) (xy 269.24 97.79))
+    (stroke (width 0) (type default) (color 0 0 0 0))
+  )
   (wire (pts (xy 83.82 33.02) (xy 83.82 35.56))
     (stroke (width 0) (type default) (color 0 0 0 0))
@@
     (stroke (width 0) (type default) (color 0 0 0 0))
   )
+  (polyline (pts (xy 266.7 107.95) (xy 271.78 107.95))
+    (stroke (width 0) (type default) (color 0 0 0 0))
+  )
   (wire (pts (xy 222.25 109.22) (xy 229.87 109.22))
     (stroke (width 0) (type default) (color 0 0 0 0))
@@
     (stroke (width 0) (type default) (color 0 0 0 0))
   )
+  (wire (pts (xy 266.7 92.71) (xy 269.24 92.71))
+    (stroke (width 0) (type default) (color 0 0 0 0))
+  )
   (wire (pts (xy 31.75 26.67) (xy 41.91 26.67))
     (stroke (width 0) (type default) (color 0 0 0 0))
@@
   )
   (text "1.8 V LDO" (at 125.73 50.8 0)
+    (effects (font (size 1.27 1.27)) (justify left bottom))
+  )
+  (text "Optional GND connectors\nfor each output" (at 259.08 113.03 0)
     (effects (font (size 1.27 1.27)) (justify left bottom))
   )
@@
     (pin "2")
   )
+  (symbol (lib_id "power:GND") (at 269.24 100.33 0) (unit 1)
+    (in_bom yes) (on_board yes) (fields_autoplaced)
+    (property "Reference" "#PWR?" (id 0) (at 269.24 106.68 0)
+      (effects (font (size 1.27 1.27)) hide)
+    )
+    (property "Value" "GND" (id 1) (at 269.24 105.41 0))
+    (property "Footprint" "" (id 2) (at 269.24 100.33 0)
+      (effects (font (size 1.27 1.27)) hide)
+    )
+    (property "Datasheet" "" (id 3) (at 269.24 100.33 0)
+      (effects (font (size 1.27 1.27)) hide)
+    )
+    (pin "1")
+  )
   (symbol (lib_id "Device:C") (at 182.88 86.36 0) (unit 1)
     (in_bom yes) (on_board yes) (fields_autoplaced)
@@
     (pin "1")
     (pin "2")
-  )
-  (symbol (lib_id "Connector:Conn_01x03_Female") (at 259.08 95.25 0) (unit 1)
-    (in_bom yes) (on_board yes) (fields_autoplaced)
-    (property "Reference" "J2" (id 0) (at 260.35 93.9799 0)
-      (effects (font (size 1.27 1.27)) (justify left))
-    )
-    (property "Value" "Conn_01x03_Female" (id 1) (at 260.35 96.5199 0)
-      (effects (font (size 1.27 1.27)) (justify left))
-    )
-    (property "Footprint" "Connector_PinSocket_2.54mm:PinSocket_1x03_P2.54mm_Vertical" (id 2) (at 259.08 95.25 0)
-      (effects (font (size 1.27 1.27)) hide)
-    )
-    (property "Datasheet" "~" (id 3) (at 259.08 95.25 0)
-      (effects (font (size 1.27 1.27)) hide)
-    )
-    (pin "1")
-    (pin "2")
-    (pin "3")
   )
   (symbol (lib_id "power:GND") (at 182.88 92.71 0) (unit 1)
@@
     )
     (pin "1")
+  )
+  (symbol (lib_id "Connector_Generic:Conn_02x03_Odd_Even") (at 259.08 95.25 0) (unit 1)
+    (in_bom yes) (on_board yes) (fields_autoplaced)
+    (property "Reference" "J?" (id 0) (at 260.35 86.36 0))
+    (property "Value" "Conn_02x03_Odd_Even" (id 1) (at 260.35 88.9 0))
+    (property "Footprint" "" (id 2) (at 259.08 95.25 0)
+      (effects (font (size 1.27 1.27)) hide)
+    )
+    (property "Datasheet" "~" (id 3) (at 259.08 95.25 0)
+      (effects (font (size 1.27 1.27)) hide)
+    )
+    (pin "1")
+    (pin "2")
+    (pin "3")
+    (pin "4")
+    (pin "5")
+    (pin "6")
   )
   (symbol (lib_id "THS8135PHP:THS8135PHP") (at 120.65 104.14 0) (unit 1)
@@
       (reference "#PWR0151") (unit 1) (value "+1V8") (footprint "")
     )
+    (path "/8566b859-6160-4a91-8ef1-06e2d1397640"
+      (reference "#PWR?") (unit 1) (value "GND") (footprint "")
+    )
     (path "/78b86417-dc5c-444f-850c-af12e2b87b9d"
       (reference "C1") (unit 1) (value "100n") (footprint "Capacitor_SMD:C_0603_1608Metric")
@@
       (reference "J1") (unit 1) (value "Conn_01x03_Female") (footprint "Connector_PinSocket_2.54mm:PinSocket_1x03_P2.54mm_Vertical")
     )
-    (path "/91b711c6-eaeb-4b1f-9eb3-e78ece718130"
-      (reference "J2") (unit 1) (value "Conn_01x03_Female") (footprint "Connector_PinSocket_2.54mm:PinSocket_1x03_P2.54mm_Vertical")
-    )
     (path "/43f72e4b-8646-4e37-984e-c6026129efb2/9a599ff9-8c2c-43a5-9985-4beb751d9c73"
       (reference "J3") (unit 1) (value "Conn_01x10_Female") (footprint "Connector_PinSocket_2.54mm:PinSocket_1x10_P2.54mm_Vertical")
@@
       (reference "J5") (unit 1) (value "Conn_01x08_Female") (footprint "Connector_PinSocket_2.54mm:PinSocket_1x08_P2.54mm_Vertical")
     )
+    (path "/da49dfaa-368b-4be0-811b-4742561422e4"
+      (reference "J?") (unit 1) (value "Conn_02x03_Odd_Even") (footprint "")
+    )
     (path "/6cdd7ab4-7b3a-4741-b4e8-e37bfc91a0a8/3b0918d9-3f04-41c3-9be9-d67031036192"

Commit message: again
Parts:
- J2: renamed from J?; footprint (none) -> Connector_PinSocket_2.54mm:PinSocket_2x03_P2.54mm_Vertical
- renumbered C7 to C5, C5 to C6, C6 to C7
