File: DAC/DAC-peripherals/level_shifter_2channel_sch.kicad_sch (KiCad schematic)
At the start: 1 part

Commit message: improved PCB again again
Parts:
- gave numbers to parts that had none: 1
Other:
- note added: "You could replace these with mosfet level-shifters, this would add a lot more components to the BOM but will overall be cheaper."
Changed lines of the file:
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@@
     (stroke (width 0) (type default) (color 0 0 0 0))
+  )
+  (text "You could replace these with mosfet level-shifters,\nthis would add a lot more components to the BOM but\nwill overall be cheaper."
+    (at 146.05 129.54 0)
+    (effects (font (size 1.27 1.27)) (justify left bottom))
   )
   (hierarchical_label "in2" (shape input) (at 158.75 91.44 0)
@@
   (symbol (lib_id "power:+1V8") (at 143.51 73.66 0) (unit 1)
     (in_bom yes) (on_board yes) (fields_autoplaced)
-    (property "Reference" "#PWR?" (id 0) (at 143.51 77.47 0)
+    (property "Reference" "#PWR0111" (id 0) (at 143.51 77.47 0)
       (effects (font (size 1.27 1.27)) hide)
     )
@@
   (symbol (lib_id "Logic_LevelTranslator:74LVC2T45DC") (at 146.05 88.9 0) (unit 1)
     (in_bom yes) (on_board yes) (fields_autoplaced)
-    (property "Reference" "U?" (id 0) (at 148.0694 101.6 0)
+    (property "Reference" "U2" (id 0) (at 148.0694 101.6 0)
       (effects (font (size 1.27 1.27)) (justify left))
     )
@@
   (symbol (lib_id "power:+3.3V") (at 148.59 73.66 0) (unit 1)
     (in_bom yes) (on_board yes) (fields_autoplaced)
-    (property "Reference" "#PWR?" (id 0) (at 148.59 77.47 0)
+    (property "Reference" "#PWR0110" (id 0) (at 148.59 77.47 0)
       (effects (font (size 1.27 1.27)) hide)
     )
@@
   (symbol (lib_id "power:GND") (at 146.05 104.14 0) (unit 1)
     (in_bom yes) (on_board yes) (fields_autoplaced)
-    (property "Reference" "#PWR?" (id 0) (at 146.05 110.49 0)
+    (property "Reference" "#PWR0109" (id 0) (at 146.05 110.49 0)
       (effects (font (size 1.27 1.27)) hide)
     )
